File: hardware/kicad/wisp.kicad_sch (KiCad schematic)
At the start: 69 parts, among them J1 USB-C, J2 Second I2C Bus, J3 mmWave UART (LD2410), J4 I2S Mic (INMP441), J5 Switched DC Output, J6 Reed/Hall Contact, J7 1-Wire Bus, J8 Analog Sensor Pad, J9 Expansion Header, Q1 MMBT3904, Q2 MMBT3904, Q3 2N7002, Q4 MMBT3904, SW1 RESET, SW2 BOOT, U1 CH340C, U2 AP63203WU-7, U3 ESP32-WROOM-32, U4 SCD41-D-R2, U5 BME680, U6 BH1750FVI-TR

Commit message: Add first-pass PCB layout, fix schematic DNP flags, prep prototype BOM/CPL
Placement for all 69 schematic parts on a 140x100mm 2-layer board,
DRC-clean (0 violations): power/USB-C/buck top-left, CH340 + auto-reset
below it, ESP32-WROOM-32 with its antenna keepout clear near the top
edge, sensor trio + I2C pull-ups center, DNP expansion headers along the
right/bottom edges, test-point cluster for bed-of-nails access. GND and
+3V3 are realized as copper pours (GND stitched with vias); the other 44
signal nets are left as ratsnest for interactive routing or a real
autorouter -- not attempted here since a naive single-layer point-to-point
router produced hundreds of shorts/crossings. Board is not fab-ready yet
(no Gerbers generated) pending that routing pass.

Also fixes three schematic DNP flags that didn't match the documented
decisions in docs/hardware-expandability.md: F1 and TP1-TP10 were marked
DNP despite being "Include" (always-populated) items, and the ESD diode
covering EXP_IO39 (D10) was missing a footprint/DNP assignment entirely.

BOM and CPL for the first physical prototype (DNP parts excluded, per the
"what gets populated" decision) are in hardware/fab/, plus a full BOM
covering every DNP option for later builds.

Co-Authored-By: Claude Sonnet 5 <noreply@anthropic.com>
Parts:
- BZ1: footprint (none) -> Buzzer_Beeper:Buzzer_CUI_CPT-9019S-SMT
- D10, D2, D3, D4, D5, D6, D7, D8, D9, F1, TP1, TP10, TP2, TP3, TP4, TP5, TP6, TP7, TP8, TP9: now fitted
Changed lines of the file:
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@@
   )
   (symbol (lib_id "Diode:PESD5V0L1UL") (at 44.45 195.58 0) (unit 1)
-    (in_bom yes) (on_board yes) (dnp yes)
+    (in_bom yes) (on_board yes)
     (property "Reference" "D2" (at 44.45 187.58 0)
       (effects (font (size 1.27 1.27)))
@@
   )
   (symbol (lib_id "Diode:PESD5V0L1UL") (at 74.93 195.58 0) (unit 1)
-    (in_bom yes) (on_board yes) (dnp yes)
+    (in_bom yes) (on_board yes)
     (property "Reference" "D3" (at 74.93 187.58 0)
       (effects (font (size 1.27 1.27)))
@@
   )
   (symbol (lib_id "Diode:1N4148") (at 224.79 177.8 0) (unit 1)
-    (in_bom yes) (on_board yes) (dnp yes)
+    (in_bom yes) (on_board yes)
     (property "Reference" "D4" (at 224.79 169.8 0)
       (effects (font (size 1.27 1.27)))
@@
       (effects (font (size 1.27 1.27)))
     )
+    (property "Footprint" "Buzzer_Beeper:Buzzer_CUI_CPT-9019S-SMT" (at 265.43 177.8 0)
+      (effects (font (size 1.27 1.27)) hide)
+    )
     (pin "1")
     (pin "2")
@@
   )
   (symbol (lib_id "Diode:PESD5V0L1UL") (at 44.45 219.71 0) (unit 1)
-    (in_bom yes) (on_board yes) (dnp yes)
+    (in_bom yes) (on_board yes)
     (property "Reference" "D5" (at 44.45 211.71 0)
       (effects (font (size 1.27 1.27)))
@@
   )
   (symbol (lib_id "Diode:PESD5V0L1UL") (at 100.33 224.79 0) (unit 1)
-    (in_bom yes) (on_board yes) (dnp yes)
+    (in_bom yes) (on_board yes)
     (property "Reference" "D6" (at 100.33 216.79 0)
       (effects (font (size 1.27 1.27)))
@@
   )
   (symbol (lib_id "Diode:PESD5V0L1UL") (at 195.58 232.41 0) (unit 1)
-    (in_bom yes) (on_board yes) (dnp yes)
+    (in_bom yes) (on_board yes)
     (property "Reference" "D7" (at 195.58 224.41 0)
       (effects (font (size 1.27 1.27)))
@@
   )
   (symbol (lib_id "Diode:PESD5V0L1UL") (at 220.98 232.41 0) (unit 1)
-    (in_bom yes) (on_board yes) (dnp yes)
+    (in_bom yes) (on_board yes)
     (property "Reference" "D8" (at 220.98 224.41 0)
       (effects (font (size 1.27 1.27)))
@@
   )
   (symbol (lib_id "Diode:PESD5V0L1UL") (at 246.38 232.41 0) (unit 1)
-    (in_bom yes) (on_board yes) (dnp yes)
+    (in_bom yes) (on_board yes)
     (property "Reference" "D9" (at 246.38 224.41 0)
       (effects (font (size 1.27 1.27)))
@@
   )
   (symbol (lib_id "Diode:PESD5V0L1UL") (at 271.78 232.41 0) (unit 1)
-    (in_bom yes) (on_board yes) (dnp yes)
+    (in_bom yes) (on_board yes)
     (property "Reference" "D10" (at 271.78 224.41 0)
       (effects (font (size 1.27 1.27)))
@@
   )
   (symbol (lib_id "Connector:TestPoint") (at 30.48 261.62 0) (unit 1)
-    (in_bom yes) (on_board yes) (dnp yes)
+    (in_bom yes) (on_board yes)
     (property "Reference" "TP1" (at 30.48 258.62 0)
       (effects (font (size 1.27 1.27)))
@@
   )
   (symbol (lib_id "Connector:TestPoint") (at 45.72 261.62 0) (unit 1)
-    (in_bom yes) (on_board yes) (dnp yes)
+    (in_bom yes) (on_board yes)
     (property "Reference" "TP2" (at 45.72 258.62 0)
       (effects (font (size 1.27 1.27)))
@@
   )
   (symbol (lib_id "Connector:TestPoint") (at 60.96 261.62 0) (unit 1)
-    (in_bom yes) (on_board yes) (dnp yes)
+    (in_bom yes) (on_board yes)
     (property "Reference" "TP3" (at 60.96 258.62 0)
       (effects (font (size 1.27 1.27)))
@@
   )
   (symbol (lib_id "Connector:TestPoint") (at 76.2 261.62 0) (unit 1)
-    (in_bom yes) (on_board yes) (dnp yes)
+    (in_bom yes) (on_board yes)
     (property "Reference" "TP4" (at 76.2 258.62 0)
       (effects (font (size 1.27 1.27)))
@@
   )
   (symbol (lib_id "Connector:TestPoint") (at 139.7 261.62 0) (unit 1)
-    (in_bom yes) (on_board yes) (dnp yes)
+    (in_bom yes) (on_board yes)
     (property "Reference" "TP5" (at 139.7 258.62 0)
       (effects (font (size 1.27 1.27)))
@@
   )
   (symbol (lib_id "Connector:TestPoint") (at 154.94 261.62 0) (unit 1)
-    (in_bom yes) (on_board yes) (dnp yes)
+    (in_bom yes) (on_board yes)
     (property "Reference" "TP6" (at 154.94 258.62 0)
       (effects (font (size 1.27 1.27)))
@@
   )
   (symbol (lib_id "Connector:TestPoint") (at 170.18 261.62 0) (unit 1)
-    (in_bom yes) (on_board yes) (dnp yes)
+    (in_bom yes) (on_board yes)
     (property "Reference" "TP7" (at 170.18 258.62 0)
       (effects (font (size 1.27 1.27)))
@@
   )
   (symbol (lib_id "Connector:TestPoint") (at 185.42 261.62 0) (unit 1)
-    (in_bom yes) (on_board yes) (dnp yes)
+    (in_bom yes) (on_board yes)
     (property "Reference" "TP8" (at 185.42 258.62 0)
       (effects (font (size 1.27 1.27)))
@@
   )
   (symbol (lib_id "Connector:TestPoint") (at 200.66 261.62 0) (unit 1)
-    (in_bom yes) (on_board yes) (dnp yes)
+    (in_bom yes) (on_board yes)
     (property "Reference" "TP9" (at 200.66 258.62 0)
       (effects (font (size 1.27 1.27)))
@@
   )
   (symbol (lib_id "Connector:TestPoint") (at 215.9 261.62 0) (unit 1)
-    (in_bom yes) (on_board yes) (dnp yes)
+    (in_bom yes) (on_board yes)
     (property "Reference" "TP10" (at 215.9 258.62 0)
       (effects (font (size 1.27 1.27)))
@@
   )
   (symbol (lib_id "Device:Polyfuse") (at 260.35 224.79 0) (unit 1)
-    (in_bom yes) (on_board yes) (dnp yes)
+    (in_bom yes) (on_board yes)
     (property "Reference" "F1" (at 260.35 216.79 0)
       (effects (font (size 1.27 1.27)))

Commit message: Rev B: ESP32-S3, open-source VOC sensing, and generated design sources
Design review of Rev A turned up a board that would not have booted, plus a
sensor choice that could not be used without a proprietary binary blob. This
rebuilds the board around both findings.

The blocker. Rev A's auto-reset circuit drove two grounded-emitter NPNs
directly from the CH340C's active-low DTR#/RTS# outputs. Those idle HIGH, so
EN was pulled low whenever the bridge was powered and RTS was not asserted --
including on a plain USB charger. The board would have sat in reset out of the
box, and esptool's sequence would have released it only while a port was open.

Rather than patch that circuit, the MCU moves to ESP32-S3-WROOM-1-N8. Native
USB deletes the CH340C, both auto-reset transistors, their resistors and
decoupling -- nine parts and the entire bug class -- and brings USB-Serial-JTAG
so debugging needs no extra connector. It also retires the WROOM-32's
flash-voltage strapping trap on IO12, since that role belongs to IO45 on the
S3, which is not broken out.

Sensors. BME680 -> SGP41 + BME280. The BME680's gas signal is only usable
through Bosch BSEC, a closed-source blob that conflicts with the MIT licence
on /firmware and with the project's "full control over the code" premise;
Sensirion's Gas Index Algorithm is BSD-3-Clause and adds NOx alongside VOC.
Dropping the BME680 would have lost barometric pressure, so the BME280 joins
it -- not as a nicety, but because the SCD41 needs ambient pressure to
compensate its CO2 reading.

Also fixed, from the same review:
- C7 100nF, not 2.2nF (AP63203 datasheet value for the bootstrap cap)
- 10uF bulk at the module's 3V3 pin; Rev A's nearest bulk was 26mm away
- 10uF at the SCD41, which draws 205mA measurement peaks
- second 22uF at the buck output, per the datasheet's 2x22uF
- SGP41 gets its datasheet RC element: 4.7R + 1uF on VDD, own 1uF on VDDH
- USBLC6-2SC6 on D+/D-/VBUS; Rev A protected the DNP headers but not USB
- 220R series resistor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
Parts:
- removed C1, C11, C8: 100nF, Capacitor_SMD:C_0805_2012Metric, symbol Device:C
- removed D4: 1N4148W, Diode_SMD:D_SOD-123, symbol Diode:1N4148
- removed J5: Switched DC Output, Connector_PinHeader_2.54mm:PinHeader_1x02_P2.54mm_Vertical, symbol Connector_Generic:Conn_01x02
- removed J9: Expansion Header, Connector_PinHeader_2.54mm:PinHeader_1x06_P2.54mm_Vertical, symbol Connector_Generic:Conn_01x06
- removed Q1, Q2: MMBT3904, Package_TO_SOT_SMD:SOT-23, symbol Transistor_BJT:MMBT3904
- removed Q3: 2N7002, Package_TO_SOT_SMD:SOT-23, symbol Transistor_FET:2N7002
- removed R5, R6: 10k, Resistor_SMD:R_0805_2012Metric, symbol Device:R
- removed U1: CH340C, Package_SO:SOIC-16_3.9x9.9mm_P1.27mm, symbol wisp:CH340C
- removed U3: ESP32-WROOM-32, RF_Module:ESP32-WROOM-32, symbol RF_Module:ESP32-WROOM-32
- removed U5: BME680, Package_LGA:Bosch_LGA-8_3x3mm_P0.8mm_ClockwisePinNumbering, symbol Sensor:BME680
- added C12, C13: 10uF, Capacitor_SMD:C_0805_2012Metric, symbol Device:C
- added C14: 22uF, Capacitor_SMD:C_0805_2012Metric, symbol Device:C
- added C16, C17, C18, C19: 100nF, Capacitor_SMD:C_0805_2012Metric, symbol Device:C
- added C20, C21: 1uF, Capacitor_SMD:C_0805_2012Metric, symbol Device:C
- added D11: 1N4148W, Diode_SMD:D_SOD-123, symbol Diode:1N4148W
- added D12: GREEN, LED_SMD:LED_0805_2012Metric, symbol Device:LED
- added D13, D14, D15: PESD5V0L1UL, Diode_SMD:D_SOD-882, symbol Diode:PESD5V0L1UL
- added D4: SS14, Diode_SMD:D_SMA, symbol Diode:SS14
- added J5: Switched DC Output, Connector_PinHeader_2.54mm:PinHeader_1x03_P2.54mm_Vertical, symbol Connector_Generic:Conn_01x03
- added J9: Expansion Header, Connector_PinHeader_2.54mm:PinHeader_1x08_P2.54mm_Vertical, symbol Connector_Generic:Conn_01x08
- added MH1, MH2, MH3, MH4: MountingHole_M3, MountingHole:MountingHole_3.2mm_M3, symbol Mechanical:MountingHole
- added Q3: AO3400A, Package_TO_SOT_SMD:SOT-23, symbol Transistor_FET:AO3400A
- added R15, R16, R17: 220R, Resistor_SMD:R_0805_2012Metric, symbol Device:R
- added R18: 100k, Resistor_SMD:R_0805_2012Metric, symbol Device:R
- added R20: 10k, Resistor_SMD:R_0805_2012Metric, symbol Device:R
- added R21: 2.2k, Resistor_SMD:R_0805_2012Metric, symbol Device:R
- added R22: 4.7R, Resistor_SMD:R_0805_2012Metric, symbol Device:R
- added TP11: UART0_TX, TestPoint:TestPoint_Pad_1.5x1.5mm, symbol Connector:TestPoint
- added TP12: UART0_RX, TestPoint:TestPoint_Pad_1.5x1.5mm, symbol Connector:TestPoint
- added TP13: LED_DOUT, TestPoint:TestPoint_Pad_1.5x1.5mm, symbol Connector:TestPoint
- added U3: ESP32-S3-WROOM-1-N8, wisp:ESP32-S3-WROOM-1, symbol RF_Module:ESP32-S3-WROOM-1
- added U5: SGP41, wisp:Sensirion_DFN-6-1EP_2.44x2.44mm_P0.8mm_EP1.25x1.7mm, symbol wisp:SGP41
- added U7: BME280, Package_LGA:Bosch_LGA-8_2.5x2.5mm_P0.65mm_ClockwisePinNumbering, symbol Sensor:BME280
- added U8: USBLC6-2SC6, Package_TO_SOT_SMD:SOT-23-6, symbol Power_Protection:USBLC6-2SC6
- BZ1: MPN (none) -> CPT-9019S-SMT; Manufacturer (none) -> CUI Devices; Rating (none) -> piezo transducer, external drive
- C10, C2, C9: MPN (none) -> CL21B104KBCNNNC; Manufacturer (none) -> Samsung; Rating (none) -> 50V X7R
- C3: MPN (none) -> CL21A106KOQNNNE; Manufacturer (none) -> Samsung; Rating (none) -> 16V X5R
- C4: MPN (none) -> CL21A105KBFNNNE; Manufacturer (none) -> Samsung; Rating (none) -> 25V X5R
- C5: MPN (none) -> CL21A106KOQNNNE; Manufacturer (none) -> Samsung; Rating (none) -> 25V X5R
- C6: MPN (none) -> CL21A226MOQNNNE; Manufacturer (none) -> Samsung; Rating (none) -> 16V X5R
- C7: value 2.2nF -> 100nF; MPN (none) -> CL21B104KBCNNNC; Manufacturer (none) -> Samsung; Rating (none) -> 50V X7R
- D1: MPN (none) -> WS2812B; Manufacturer (none) -> Worldsemi; Rating (none) -> VDD 3.5-5.3V
- D10, D2, D3, D5, D6, D7, D8, D9: MPN (none) -> PESD5V0L1UL; Manufacturer (none) -> Nexperia
- F1: MPN (none) -> MF-MSMF050-2; Manufacturer (none) -> Bourns; Rating (none) -> PTC, 500mA hold, 6V
- J1: MPN (none) -> TYPE-C-31-M-12; Manufacturer (none) -> HRO
- L1: MPN (none) -> SRN3015-2R2M; Manufacturer (none) -> Bourns; Rating (none) -> Isat >= 1.5A, DCR < 100mOhm
- Q4: MPN (none) -> MMBT3904; Manufacturer (none) -> onsemi
- R1, R2: MPN (none) -> RC0805FR-075K1L; Manufacturer (none) -> Yageo; Rating (none) -> 1%, 1/8W
- R10, R11: MPN (none) -> RC0805FR-074K7L; Manufacturer (none) -> Yageo; Rating (none) -> 1%
- R12: MPN (none) -> RC0805FR-07100RL; Manufacturer (none) -> Yageo; Rating (none) -> 1%, gate series
- R13: MPN (none) -> RC0805FR-071KL; Manufacturer (none) -> Yageo; Rating (none) -> 1%, base series
- R14: MPN (none) -> RC0805FR-074K7L; Manufacturer (none) -> Yageo; Rating (none) -> 1%, 1-Wire pull-up
- R3, R4: MPN (none) -> RC0805FR-0710KL; Manufacturer (none) -> Yageo; Rating (none) -> 1%, 1/8W
- R7: MPN (none) -> RC0805FR-07330RL; Manufacturer (none) -> Yageo; Rating (none) -> 1%, 1/8W
- R8, R9: MPN (none) -> RC0805FR-074K7L; Manufacturer (none) -> Yageo; Rating (none) -> 1%, I2C pull-up
- SW1, SW2: MPN (none) -> PTS810 SJM 250 SMTR LFS; Manufacturer (none) -> C&K
- TP1: value JTAG_TDI -> JTAG_MTDI
- TP2: value JTAG_TCK -> JTAG_MTCK
- TP3: value JTAG_TMS -> JTAG_MTMS
- TP4: value JTAG_TDO -> JTAG_MTDO
- U2: MPN (none) -> AP63203WU-7; Manufacturer (none) -> Diodes Incorporated; Rating (none) -> 2A sync buck, fixed 3.3V
- U4: MPN (none) -> SCD41-D-R2; Manufacturer (none) -> Sensirion; Rating (none) -> CO2/T/RH, I2C 0x62
- U6: MPN (none) -> BH1750FVI-TR; Manufacturer (none) -> ROHM; Rating (none) -> lux, I2C 0x23
Connections:
- net +3V3: now also C12.1, C13.1, C14.1, C18.1, C19.1, C21.1, J9.2 (Pin_2), R21.1, R22.1, U3.2 (3V3), U5.5 (VDDH), U7.2 (CSB), U7.6 (VDDIO), U7.8 (VDD); no longer D1.1 (VDD)
- net +5V: now also U8.5 (VBUS)
- net +5V_EXT: now also D11.2 (A), D4.1 (K), J5.1 (Pin_1)
- net ADC_PAD: now also C16.1, R17.2, U3.4 (IO4); no longer J8.3 (Pin_3)
- net BUZZER_CTRL: now also U3.8 (IO15)
- net EN: now also U3.3 (EN)
- net GND: now also C12.2, C13.2, C14.2, C16.2, C17.2, C18.2, C19.2, C20.2, C21.2, D12.1 (K), D13.2 (A), D14.2 (A), D15.2 (A), J5.3 (Pin_3), J9.1 (Pin_1), Q3.2 (S), R18.2, R20.2, U3.1 (GND), U3.40 (GND), U3.41 (GND), U5.2 (VSS), U5.4 (NC_GND), U5.7 (EP), U7.1 (GND), U7.5 (SDO), U7.7 (GND), U8.2 (GND)
- net IO0: now also U3.27 (IO0)
- net LED_CTRL: now also R20.1, U3.7 (IO7)
- net MIC_SCK: now also U3.20 (IO12)
- net MIC_SD: now also U3.22 (IO14)
- net MIC_WS: now also U3.21 (IO13)
- net MMWAVE_RX: now also U3.18 (IO10)
- net MMWAVE_TX: now also U3.19 (IO11)
- net ONEWIRE_DATA: now also R16.2, U3.5 (IO5); no longer D6.1 (K), J7.3 (Pin_3), R14.2
- net REED_IN: now also R15.2, U3.6 (IO6); no longer D5.1 (K), J6.1 (Pin_1)
- net SCL: now also U3.17 (IO9), U5.6 (SCL), U7.4 (SCK)
- net SCL2: now also U3.11 (IO18)
- net SDA: now also U3.12 (IO8), U5.3 (SDA), U7.3 (SDI)
- net SDA2: now also U3.10 (IO17)
- net SW_GND: now also D4.2 (A), J5.2 (Pin_2), Q3.3 (D)
- net SW_OUT_CTRL: now also U3.9 (IO16)
- net SW_OUT_GATE: now also Q3.1 (G), R18.1
- net USB_DM: now also U3.13 (USB_D-), U8.1 (I/O1), U8.6 (I/O1)
- net USB_DP: now also U3.14 (USB_D+), U8.3 (I/O2), U8.4 (I/O2)
- net LED_DOUT: now reaches D1.2 (DOUT)
- net LED_DOUT: now also TP13.1
- net EXP_IO33 renamed EXP_IO1
- net EXP_IO1: now also J9.3 (Pin_3), U3.39 (IO1)
- net EXP_IO34 renamed EXP_IO2
- net EXP_IO2: now also J9.4 (Pin_4), U3.38 (IO2)
- net EXP_IO35 renamed EXP_IO21
- net EXP_IO21: now also J9.5 (Pin_5), U3.23 (IO21)
- net EXP_IO39 renamed EXP_IO38
- net EXP_IO38: now also J9.6 (Pin_6), U3.31 (IO38)
- net JTAG_TCK renamed JTAG_MTCK
- net JTAG_MTCK: now also U3.32 (IO39)
- net JTAG_TDI renamed JTAG_MTDI
- net JTAG_MTDI: now also U3.34 (IO41)
- net JTAG_TDO renamed JTAG_MTDO
- net JTAG_MTDO: now also U3.33 (IO40)
- net JTAG_TMS renamed JTAG_MTMS
- net JTAG_MTMS: now also U3.35 (IO42)
- new net ADC_PAD_EXT: D13.1 (K), J8.3 (Pin_3), R17.1
- new net EXP_IO47: D14.1 (K), J9.7 (Pin_7), U3.24 (IO47)
- new net EXP_IO48: D15.1 (K), J9.8 (Pin_8), U3.25 (IO48)
- new net LED_VCC: C17.1, D1.1 (VDD), D11.1 (K)
- new net ONEWIRE_EXT: D6.1 (K), J7.3 (Pin_3), R14.2, R16.1
- new net PWR_LED: D12.2 (A), R21.2
- new net REED_EXT: D5.1 (K), J6.1 (Pin_1), R15.1
- new net SGP_VDD: C20.1, R22.2, U5.1 (VDD)
- new net UART0_RX: TP12.1, U3.36 (RXD0)
- new net UART0_TX: TP11.1, U3.37 (TXD0)
- no-connect marks 15 -> 8
Other:
- note added: "5V -> 3V3 buck regulator"
- note added: "DNP expansion footprints (see docs/hardware-expandability.md)"
- note added: "ESP32-S3-WROOM-1 (native USB, no UART bridge)"
- note added: "Mounting holes"
- note added: "Sensors: SCD41 CO2/T/RH, SGP41 VOC/NOx, BME280 pressure, BH1750 lux"
- note added: "Status LED (WS2812B on ~4.3V) + power-on LED"
- note added: "Test points"
- note added: "USB-C input, ESD protection, PTC fuse"
- note removed: "-- DNP expansion footprints below (see docs/hardware-expandability.md) --"
- note removed: "1-Wire bus pad (e.g. DS18B20)"
- note removed: "Analog sensor pad (ADC1-capable)"
- note removed: "General test points (factory test / recovery flashing)"
- note removed: "Generic expansion header (spare GPIO, also ADC1-capable)"
- note removed: "I2S microphone header (INMP441)"
- note removed: "JTAG test points (MTDI/MTCK/MTMS/MTDO, pads only)"
- note removed: "PTC fuse for externally-exposed 5V pins"
- note removed: "Piezo buzzer (local alarm)"
- note removed: "Reed/Hall contact pad (window sensor)"
- note removed: "Second I2C bus (isolated, own pull-ups)"
- note removed: "Switched DC output (low-voltage only, DC fan/dehumidifier)"
- note removed: "mmWave presence UART header (LD2410)"

Commit message: Verify BH1750 footprint, add LCSC numbers, fix JLCPCB DFM findings
Closes the items left open from PR #11 (issue #12):

- wisp:BH1750FVI-TR_WSOF6 is no longer a DRAFT footprint. ROHM's
  mechanical drawing (Technical Note No.11046EDT01 Rev.D, p.14) turned
  out to be reachable; the land pattern is rebuilt from its figures and
  cross-checked against the LCSC C78960 listing. The exposed centre pad
  is copper-only, no paste, no net, per the datasheet's explicit
  "do not solder" note on that pad.
- LCSC part numbers added for 27 of 33 unique BOM parts, each verified
  against its LCSC catalogue page (manufacturer + MPN + package), not
  guessed. Six are deliberately left blank (not stocked, ambiguous
  variant, or only in JLCPCB's Extended Parts Library) -- see the
  hardware README for the list and why.
- F1's footprint was Fuse_1206_3216Metric; MF-MSMF050-2 is actually a
  1812 part. Caught while verifying its LCSC entry, fixed to
  Fuse_1812_4532Metric.
- SGP41 soldering guidance in the README expanded with the exact
  reflow profile from Sensirion's datasheet (no-clean type 3 paste,
  245C/30s peak, no hand/vapour-phase soldering, no board wash).

Also fixed what a JLCPCB DFM report found that local DRC couldn't see,
because wisp.kicad_dru carried no rules and min_silk_clearance /
solder_mask_to_copper_clearance were both 0 in wisp.kicad_pro:

- Root cause of the silkscreen findings was in gen_pcb.py's silk
  stage: reference-designator placement estimated each label's size
  from a 0.62mm/character formula instead of querying KiCad's real
  rendered bounding box, undershooting it by up to 0.48mm, and never
  considered vias as obstacles at all. Both fixed -- the search now
  reads GetBoundingBox() off the actual text object and indexes vias
  alongside pads. Verified directly: silk-to-via and silk-to-pad
  clearance violations under 0.15mm went from 35 and 117 to 0.
- wisp.kicad_pro rules now match JLCPCB's published capability
  (min_silk_clearance 0.15mm, sold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
Parts:
- BZ1: LCSC (none) -> C95163
- C10, C16, C17, C18, C19, C2, C7, C9: LCSC (none) -> C1711
- C12, C13, C3, C5: LCSC (none) -> C1713
- C14, C6: LCSC (none) -> C98190
- D10, D13, D14, D15, D2, D3, D5, D6, D7, D8, D9: LCSC (none) -> C552556
- D11: LCSC (none) -> C83528
- F1: footprint Fuse:Fuse_1206_3216Metric -> Fuse:Fuse_1812_4532Metric; LCSC (none) -> C17313
- J1: LCSC (none) -> C165948
- L1: LCSC (none) -> C2041716
- Q3: LCSC (none) -> C20917
- Q4: LCSC (none) -> C81464
- R1, R2: LCSC (none) -> C84375
- R10, R11, R14, R8, R9: LCSC (none) -> C60816
- R12: LCSC (none) -> C105577
- R13: LCSC (none) -> C95781
- R15, R16, R17: LCSC (none) -> C114519
- R18: LCSC (none) -> C96346
- R20, R3, R4: LCSC (none) -> C84376
- R21: LCSC (none) -> C114561
- R22: LCSC (none) -> C137513
- R7: LCSC (none) -> C105878
- SW1, SW2: LCSC (none) -> C116501
- U2: LCSC (none) -> C780769
- U3: LCSC (none) -> C2913198
- U6: LCSC (none) -> C78960
- U7: LCSC (none) -> C92489
