File: hardware/kicad/wisp.kicad_pcb (KiCad board)
At the start: 2 copper layers, 140 x 100 mm, 73 parts, among them J1 USB-C, J2 Second I2C Bus, J3 mmWave UART (LD2410), J4 I2S Mic (INMP441), J5 Switched DC Output, J6 Reed/Hall Contact, J7 1-Wire Bus, J8 Analog Sensor Pad, J9 Expansion Header, Q1 MMBT3904, Q2 MMBT3904, Q3 2N7002, Q4 MMBT3904, SW1 RESET, SW2 BOOT, U1 CH340C, U2 AP63203WU-7, U3 ESP32-WROOM-32, U4 SCD41-D-R2, U5 BME680, U6 BH1750FVI-TR

Commit message: Close the U5 (+3V3) routing gap left by the last layout pass
Pin 2 of U5 (BME680) was boxed into a fully enclosed pocket on the top
layer by its own footprint's 0.8mm pitch neighbors. Turned out worse
than documented: the bottom layer was blocked at the same spot too, by
an unrelated /SW_OUT_CTRL trace (R12 to U3 pin 31) crossing directly
underneath.

Fix: local dogleg in /SW_OUT_CTRL to clear U5's footprint and escape
halo (no other constraints along that run), then a via-drop tunnel
from pin 2, under U5 on the bottom layer, back up to pin 8 (same
+3V3 net). DRC clean, 0 violations. Gerbers/drill regenerated.
Routing:
- net +3V3: track 243.9 -> 246.4 mm, vias 26 -> 28
- net /SW_OUT_CTRL: track 85.9 -> 87.2 mm
Changed lines of the file:
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@@
 	)
 	(segment
+		(start 60.9 72.8)
+		(end 60.8 73.1875)
+		(width 0.2)
+		(layer "F.Cu")
+		(net "+3V3")
+	)
+	(segment
 		(start 61.35 73.85)
 		(end 61.25 73.85)
@@
 	)
 	(via
+		(at 61.6 70.8125)
+		(size 0.6)
+		(drill 0.3)
+		(layers "F.Cu" "B.Cu")
+		(net "+3V3")
+	)
+	(via
 		(at 69.75 35.65)
 		(size 0.6)
@@
 	)
 	(via
+		(at 60.9 72.8)
+		(size 0.6)
+		(drill 0.3)
+		(layers "F.Cu" "B.Cu")
+		(net "+3V3")
+	)
+	(via
 		(at 79.098974 73.555224)
 		(size 0.6)
@@
 	)
 	(segment
+		(start 61.6 70.8125)
+		(end 60.9 72.8)
+		(width 0.2)
+		(layer "B.Cu")
+		(net "+3V3")
+	)
+	(segment
 		(start 55.15 67.85)
 		(end 55.05 67.95)
@@
 	)
 	(segment
+		(start 66 68)
+		(end 76.833 55.306)
+		(width 0.2)
+		(layer "B.Cu")
+		(net "/SW_OUT_CTRL")
+	)
+	(segment
 		(start 87.7601 38.6824)
 		(end 88.6595 38.6824)
@@
 	)
 	(segment
+		(start 48.456 83.683)
+		(end 58 78)
+		(width 0.2)
+		(layer "B.Cu")
+		(net "/SW_OUT_CTRL")
+	)
+	(segment
+		(start 62 75)
+		(end 62.2 71.5)
+		(width 0.2)
+		(layer "B.Cu")
+		(net "/SW_OUT_CTRL")
+	)
+	(segment
 		(start 76.8332 55.3059)
 		(end 76.8332 49.6093)
@@
 	)
 	(segment
-		(start 48.4563 83.6828)
-		(end 76.8332 55.3059)
+		(start 58 78)
+		(end 62 75)
 		(width 0.2)
 		(layer "B.Cu")
@@
 		(width 0.2)
 		(layer "B.Cu")
+		(net "/SW_OUT_CTRL")
+	)
+	(segment
+		(start 62.2 71.5)
+		(end 66 68)
+		(width 0.2)
+		(layer "B.Cu")
